Commit message: Working gripper implemented

File: src/ur5e_checkers_bringup/ur5e_checkers_bringup/urdf/robotiq_gripper.ros2_control.xacro (robot description, xacro)
@@ -64,5 +64,5 @@
                     <param name="multiplier">-1</param>
                     <xacro:unless value="${sim_ignition}">
-                        <command_interface name="position"/>
+                        <!-- <command_interface name="position"/> -->
                         <state_interface name="position"/>
                         <state_interface name="velocity"/>
@@ -73,5 +73,5 @@
                     <param name="multiplier">1</param>
                     <xacro:unless value="${sim_ignition}">
-                        <command_interface name="position"/>
+                        <!-- <command_interface name="position"/> -->
                         <state_interface name="position"/>
                         <state_interface name="velocity"/>
@@ -82,5 +82,5 @@
                     <param name="multiplier">-1</param>
                     <xacro:unless value="${sim_ignition}">
-                        <command_interface name="position"/>
+                        <!-- <command_interface name="position"/> -->
                         <state_interface name="position"/>
                         <state_interface name="velocity"/>
@@ -91,5 +91,5 @@
                     <param name="multiplier">-1</param>
                     <xacro:unless value="${sim_ignition}">
-                        <command_interface name="position"/>
+                        <!-- <command_interface name="position"/> -->
                         <state_interface name="position"/>
                         <state_interface name="velocity"/>
@@ -100,5 +100,5 @@
                     <param name="multiplier">1</param>
                     <xacro:unless value="${sim_ignition}">
-                        <command_interface name="position"/>
+                        <!-- <command_interface name="position"/> -->
                         <state_interface name="position"/>
                         <state_interface name="velocity"/>

File: src/ur5e_checkers_bringup/ur5e_checkers_bringup/urdf/ur5e_gripper.urdf.xacro (robot description, xacro)
@@ -1,5 +1,56 @@
 <?xml version="1.0"?>
 <robot xmlns:xacro="http://www.ros.org/wiki/xacro" name="ur5e">
-  <xacro:include filename="$(find ur_description)/urdf/ur.urdf.xacro"/>
+  <!-- =========================
+       Arguments
+       ========================= -->
+  <xacro:arg name="name" default="ur5e"/>
+  <xacro:arg name="ur_type" default="ur5e"/>
+  <xacro:arg name="tf_prefix" default=""/>
+  <!-- UR description parameters -->
+  <xacro:arg name="joint_limit_params"
+             default="$(find ur_description)/config/$(arg ur_type)/joint_limits.yaml"/>
+  <xacro:arg name="kinematics_params"
+             default="$(find ur_description)/config/$(arg ur_type)/default_kinematics.yaml"/>
+  <xacro:arg name="physical_params"
+             default="$(find ur_description)/config/$(arg ur_type)/physical_parameters.yaml"/>
+  <xacro:arg name="visual_params"
+             default="$(find ur_description)/config/$(arg ur_type)/visual_parameters.yaml"/>
+  <!-- Safety -->
+  <xacro:arg name="safety_limits" default="false"/>
+  <xacro:arg name="safety_pos_margin" default="0.15"/>
+  <xacro:arg name="safety_k_position" default="20"/>
+  <!-- Simulation / gripper -->
+  <xacro:arg name="use_fake_hardware" default="false"/>
+  <xacro:arg name="com_port" default="/dev/ttyUSB0"/>
+  <xacro:arg name="sim_gazebo" default="true"/>
+  <!-- =========================
+       Includes
+       ========================= -->
+  <xacro:include filename="$(find ur_description)/urdf/ur_macro.xacro"/>
+  <xacro:include filename="$(find ur5e_checkers_bringup)/urdf/robotiq_gripper_macro.xacro"/>
+  <!-- =========================
+       World link
+       ========================= -->
+  <link name="world"/>
+  <!-- =========================
+       UR5e arm geometry/joints
+       ========================= -->
+  <xacro:ur_robot
+      name="$(arg name)"
+      tf_prefix="$(arg tf_prefix)"
+      parent="world"
+      joint_limits_parameters_file="$(arg joint_limit_params)"
+      kinematics_parameters_file="$(arg kinematics_params)"
+      physical_parameters_file="$(arg physical_params)"
+      visual_parameters_file="$(arg visual_params)"
+      safety_limits="$(arg safety_limits)"
+      safety_pos_margin="$(arg safety_pos_margin)"
+      safety_k_position="$(arg safety_k_position)"
+      force_abs_paths="false">
+    <origin xyz="0 0 0" rpy="0 0 0"/>
+  </xacro:ur_robot>
+  <!-- =========================
+       Arm ros2_control
+       ========================= -->
   <ros2_control name="GazeboSystem" type="system">
     <hardware>
@@ -37,19 +88,25 @@
     </joint>
   </ros2_control>
-<!-- Gazebo Plugins -->
+  <!-- =========================
+       Gazebo plugin for ros2_control
+       ========================= -->
   <gazebo>
     <plugin
       filename="libgz_ros2_control-system.so"
       name="gz_ros2_control::GazeboSimROS2ControlPlugin">
-      <parameters>/workspaces/ur5e-checkers-irl/src/ur5e_checkers_bringup/ur5e_checkers_bringup/config/controllers_gripper.yaml</parameters>
+      <parameters>$(find ur5e_checkers_bringup)/config/controllers_gripper.yaml</parameters>
     </plugin>
   </gazebo>
-    <xacro:arg name="use_fake_hardware" default="false" />
-    <xacro:arg name="com_port" default="/dev/ttyUSB0" />
-    <xacro:arg name="sim_gazebo" default="true"/>
-<!-- Import macros -->
-    <xacro:include filename="$(find ur5e_checkers_bringup)/urdf/robotiq_gripper_macro.xacro" />
-    <xacro:robotiq_gripper name="RobotiqGripperHardwareInterface" prefix="" parent="tool0" use_fake_hardware="$(arg use_fake_hardware)" com_port="$(arg com_port)" sim_gazebo="$(arg sim_gazebo)">
-        <origin xyz="0 0 0" rpy="0 0 0" />
-    </xacro:robotiq_gripper>
+  <!-- =========================
+       Robotiq gripper
+       ========================= -->
+  <xacro:robotiq_gripper
+      name="RobotiqGripperHardwareInterface"
+      prefix=""
+      parent="tool0"
+      use_fake_hardware="$(arg use_fake_hardware)"
+      com_port="$(arg com_port)"
+      sim_gazebo="$(arg sim_gazebo)">
+    <origin xyz="0 0 0" rpy="0 0 0"/>
+  </xacro:robotiq_gripper>
 </robot>
